File: Hardware/Power.kicad_sch (KiCad schematic)
At the start: 16 parts, among them U1 RT9080-3.3, U4 AP7361C-3.3V

Commit message: Routing WIP
Parts:
- added VBATT.1: ~, SparkFun-Jumper:Jumper_2_NC_Trace, symbol SparkFun-Jumper:SolderJumper_2_Bridged
Connections:
- net VBATT: now also VBATT.1.2 (B); no longer C21.1, C22.1, U1.5 (VOUT)
- new net: C21.1, C22.1, U1.5 (VOUT), VBATT.1.1 (A)
Other:
- moved on the sheet: C16, C17, C18, C19, C20, C21, C22

Commit message: Updates after proto review
Parts:
- renumbered VBATT.1 to VBACKUP.1
Connections:
- net VBATT renamed VBACKUP
Other:
- note added: "Open jumper when connecting external battery or power"
- moved on the sheet: VBACKUP.1
Changed lines of the file:
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@@
+		)
+	)
+	(text "Open jumper when\nconnecting external\nbattery or power"
+		(exclude_from_sim no)
+		(at 240.03 33.02 0)
+		(effects
+			(font
+				(size 1.27 1.27)
+			)
 		)
 	)
@@
 	(wire
 		(pts
-			(xy 254 40.64) (xy 254 39.37)
+			(xy 255.27 40.64) (xy 255.27 39.37)
 		)
 		(stroke
@@
 	(wire
 		(pts
-			(xy 241.3 40.64) (xy 246.38 40.64)
+			(xy 241.3 40.64) (xy 245.11 40.64)
 		)
 		(stroke
@@
 	(wire
 		(pts
-			(xy 251.46 40.64) (xy 254 40.64)
+			(xy 250.19 40.64) (xy 255.27 40.64)
 		)
 		(stroke
@@
 	(symbol
 		(lib_id "SparkFun-Jumper:SolderJumper_2_Bridged")
-		(at 248.92 40.64 0)
+		(at 247.65 40.64 0)
 		(unit 1)
 		(exclude_from_sim no)
@@
 		(on_board yes)
 		(dnp no)
-		(property "Reference" "VBATT.1"
-			(at 248.92 38.1 0)
+		(property "Reference" "VBACKUP.1"
+			(at 247.65 38.1 0)
 			(effects
 				(font
@@
 		)
 		(property "Value" "~"
-			(at 248.92 38.1 0)
+			(at 247.65 38.1 0)
 			(effects
 				(font
@@
 		)
 		(property "Footprint" "SparkFun-Jumper:Jumper_2_NC_Trace"
-			(at 248.666 45.212 0)
+			(at 247.396 45.212 0)
 			(effects
 				(font
@@
 		)
 		(property "Datasheet" "~"
-			(at 248.92 48.26 0)
+			(at 247.65 48.26 0)
 			(effects
 				(font
@@
 		)
 		(property "Description" "Solder Jumper, 2-pole, closed/bridged"
-			(at 248.92 50.8 0)
+			(at 247.65 50.8 0)
 			(effects
 				(font
@@
 			(project ""
 				(path "/e3dd3ae4-244d-4cba-9cca-5d2abf83f29a/1cdefb16-dd9e-4f95-a59c-bf1818ce1464"
-					(reference "VBATT.1")
+					(reference "VBACKUP.1")
 					(unit 1)
 				)
@@
 	(symbol
 		(lib_id "SparkFun-PowerSymbol:VBATT")
-		(at 254 39.37 0)
+		(at 255.27 39.37 0)
 		(unit 1)
 		(exclude_from_sim no)
@@
 		(fields_autoplaced yes)
 		(property "Reference" "#PWR03"
-			(at 254 43.18 0)
-			(effects
-				(font
-					(size 1.27 1.27)
-				)
-				(hide yes)
-			)
-		)
-		(property "Value" "VBATT"
-			(at 254 35.56 0)
+			(at 255.27 43.18 0)
+			(effects
+				(font
+					(size 1.27 1.27)
+				)
+				(hide yes)
+			)
+		)
+		(property "Value" "VBACKUP"
+			(at 255.27 35.56 0)
 			(do_not_autoplace yes)
 			(effects
@@
 		)
 		(property "Footprint" ""
-			(at 254 39.37 0)
+			(at 255.27 39.37 0)
 			(effects
 				(font
@@
 		)
 		(property "Datasheet" ""
-			(at 254 39.37 0)
+			(at 255.27 39.37 0)
 			(effects
 				(font
@@
 		)
 		(property "Description" "Power symbol creates a global label with name \"VBATT\""
-			(at 254 45.72 0)
-			(effects
-				(font
+			(at 255.27 45.72 0)
+			(effects
+				(font

Commit message: PCB v02 - with corrected regulator footprint
Parts:
- U4: footprint SparkFun-Semiconductor-Standard:DFN-8_3x3mm -> SparkFun-Semiconductor-Standard:DFN-8_3x3mm_P0.65mm_EP2.25x1.5mm
Connections:
- now unconnected: U4.2 (NC), U4.3 (NC), U4.6 (NC), U4.7 (NC)
Changed lines of the file:
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@@
 			)
 		)
-		(property "Footprint" "SparkFun-Semiconductor-Standard:DFN-8_3x3mm"
+		(property "Footprint" "SparkFun-Semiconductor-Standard:DFN-8_3x3mm_P0.65mm_EP2.25x1.5mm"
 			(at 125.73 57.15 0)
 			(effects
